File: Hardware/avr-smt-44/avr-smt-44.kicad_pcb (KiCad board)
At the start: 2 copper layers, 25.4 x 72.4 mm, 31 parts, among them J1 AVR-ISP-6, SW1 SW_Push, U1 ATtiny84A-SS

Commit message: New THT version
Parts:
- added REF**: PinHeader_1x02_P2.54mm_Vertical, Connector_PinHeader_2.54mm:PinHeader_1x02_P2.54mm_Vertical, F.Cu at (172.7, 119.6)
Other:
- board text added: "EDGE CLEARANCE .040 IN"
